Commit message: add stl for belt finger, modify urdf

File: src/pb_robot/models/franka_description/robots/panda_arm_hand.urdf (robot description, URDF)
Before this commit: robot panda, 13 links, 12 joints
Links:
- link panda_leftfinger: geometry collision mesh filename=package://franka_description/meshes/collision/belt_finger_s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; visual mesh filename=package://franka_description/meshes/collision/belt_finger_s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
- link panda_rightfinger: geometry collision mesh filename=package://franka_description/meshes/collision/belt_finger_s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; visual mesh filename=package://franka_description/meshes/collision/belt_finger_s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
Joints:
- joint panda_finger_joint1: origin xyz=0 0 0.0584 rpy=0 0 0 -> xyz=0 0 0.0685 rpy=0 0 0
- joint panda_finger_joint2: origin xyz=0 0 0.0584 rpy=0 0 0 -> xyz=0 0 0.0685 rpy=0 0 0
